Commit message: tf tree aangepast, laser_link, imu_link

File: wheeltec_robot_urdf/wheeltec_robot_urdf/urdf/senior_akm_robot.urdf (robot description, URDF)
Before this commit: robot senior_akm_robot, 8 links, 7 joints
Joints:
- joint laser_joint: origin xyz=0.0887405189187401 0.000667202411597726 0.111024183741431 rpy=0 0 3.14159265358979 -> xyz=0.0887405189187401 0.000667202411597726 0.111024183741431 rpy=0 0 0
